File: board/due-pro-logic/full-board/kim1-earthpeople.kicad_pcb (KiCad board)
At the start: 2 copper layers, 116 x 53.3 mm, 10 parts, among them J101 Conn_02x18_Odd_Even, J102 Conn_02x20_Odd_Even, P2 Power, P3 XIO_4, P4 XIO_2, P5 XIO_1, P6 XIO_3, P7 XIO_5

Commit message: Version 1 of EarthPeople boards ordered.
Other:
- board text removed: "set_location_assignment PIN_55 -to PB[0]r set_location_assignment PIN_54 -to PB[1]r set_location_assignment PIN_67 -to PB[2]r set_location_assignment PIN_66 -to PB[3]r set_location_assignment PIN_53 -to PB[4]r set_location_assignment PIN_52 -to PB[5]r set_location_assignment PIN_121 -to PB[6]r set_location_assignment PIN_124 -to PB[7]r set_location_assignment PIN_120 -to AUDIOOr set_location_assi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"
Changed lines of the file:
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@@
-    (effects (font (size 1 1) (thickness 0.15)))
-  )
-  (gr_text "set_location_assignment PIN_55 -to PB[0]\r\nset_location_assignment PIN_54 -to PB[1]\r\nset_location_assignment PIN_67 -to PB[2]\r\nset_location_assignment PIN_66 -to PB[3]\r\nset_location_assignment PIN_53 -to PB[4]\r\nset_location_assignment PIN_52 -to PB[5]\r\nset_location_assignment PIN_121 -to PB[6]\r\nset_location_assignment PIN_124 -to PB[7]\r\nset_location_assignment PIN_120 -to AUDIOO\r\nset_location_assignment PIN_119 -to AUDIOI\r\n" (at 98.298 87.122) (layer "F.SilkS")
     (effects (font (size 1 1) (thickness 0.15)))
   )
